File: OpenBCI Cyton kikad Design/Cyton/Cyton.kicad_pcb (KiCad board)
At the start: 2 copper layers, 2 parts, among them IC1 ADS1299

Commit message: in-progress designs
Parts:
- added MOD1: BMD-300-A-R, digikey-footprints:Bluetooth_Module_BMD-300, F.Cu at (34.3, 40.6)
- moved IC1 1.80 mm to (29.2, 25.4)
Connections:
- net Net-(BT1-Pad2) renamed GND
